Commit message: refactored demo code, fixed launch files

File: lwr_descartes/lwr_robot/models/full_lwr/full_lwr.urdf.xacro (robot description, xacro)
@@ -13,10 +13,17 @@
         <origin xyz="0 0 0.0445" rpy="${3.1415926/2} 0 0"/>
     </xacro:robotiq_hand>
+    <!--Experimental Plugins (uncomment as needed) -->
     <gazebo>
         <plugin filename="libRobotiqHandPlugin.so" name="robotiq_controller">
             <side>left</side>
-            <kp_position>8</kp_position>
+            <kp_position>15</kp_position>
             <robotName>full_lwr</robotName>
         </plugin>
+        <!--<plugin filename="libgazebo_ros_moveit_planning_scene.so" name="gazebo_ros_moveit_planning_scene">
+            <exclude>ground_plane washer_0 washer_1</exclude>
+            <sceneName>scene</sceneName>
+            <robotName>lwr_robot</robotName>
+            <updatePeriod>0.5</updatePeriod>
+        </plugin>-->
     </gazebo>
 </robot>

File: lwr_descartes/lwr_robot/models/lwr_robot/lwr_robot.urdf.xacro (robot description, xacro)
@@ -3,7 +3,22 @@
 <robot xmlns:xacro="http://www.ros.org/wiki/xacro" name="lwr_robot">
     <xacro:include filename="$(find lwr_description)/model/kuka_lwr.urdf.xacro"/>
-    <link name="base"/>
-    <xacro:kuka_lwr parent="base" name="lwr">
+    <link name="world"/>
+    <xacro:kuka_lwr parent="world" name="lwr">
         <origin xyz="0 0 0" rpy="0 0 0"/>
     </xacro:kuka_lwr>
+    <!-- Experimental Plugins (Uncomment as needed) -->
+    <gazebo>
+        <!--<plugin name="EESwapPlugin" filename="libEESwapPlugin.so">
+                <ee_uri>
+                model://lwr_robot/models/soft_hand
+                </ee_uri>
+				<robotNamespace>lwr</robotNamespace>
+        </plugin>-->
+        <!--<plugin filename="libgazebo_ros_moveit_planning_scene.so" name="gazebo_ros_moveit_planning_scene">
+            <exclude>ground_plane washer_0 washer_1</exclude>
+            <sceneName>scene</sceneName>
+            <robotName>lwr_robot</robotName>
+            <updatePeriod>0.5</updatePeriod>
+        </plugin>-->
+    </gazebo>
 </robot>

File: lwr_descartes/lwr_robot/models/robotiq_hand/robotiq_hand.urdf.xacro (robot description, xacro)
@@ -4,5 +4,5 @@
     <link name="EE_LINK"/>
     <xacro:robotiq_hand prefix="l_" reflect="-1" parent="EE_LINK">
-        <origin xyz="0 0 0" rpy="${3.1415926/2} 0 0"/>
+        <origin xyz="0 0 0.0445" rpy="${3.1415926/2} 0 0"/>
     </xacro:robotiq_hand>
 </robot>
